File: iot-risk-data-logger-saml11.kicad_sch (KiCad schematic)
At the start: 37 parts, among them J1 Pickit 5 Conn, Q1 IRLML6401, U1 ATSAML11E16A-AU, U2 MMA8452QR1, U3 ST25DV04K, U4 OPT3001DNPR, U5 SHT30-DIS, U6 AT25SF041B-SSHD-T

Commit message: DRAFT:replace saml11 by stm32l412, add USB
Parts:
- removed J1: Pickit 5 Conn, Connector_PinSocket_2.54mm:PinSocket_1x08_P2.54mm_Vertical, symbol Connector:Conn_01x08_Socket
- removed U1: ATSAML11E16A-AU, Package_QFP:TQFP-32_7x7mm_P0.8mm, symbol ATSAML11E16A-MU:ATSAML11E16A-MU
- added C17, C18: 22p, Capacitor_SMD:C_0805_2012Metric_Pad1.18x1.45mm_HandSolder, symbol Device:C
- added C19: 4n7, Capacitor_SMD:C_0805_2012Metric_Pad1.18x1.45mm_HandSolder, symbol Device:C
- added C20: 10u, Capacitor_SMD:C_0805_2012Metric_Pad1.18x1.45mm_HandSolder, symbol Device:C
- added D2: BAT60A, Diode_SMD:D_SOD-323_HandSoldering, symbol Diode:BAT60A
- added D3: PRTR5V0U2X, Package_TO_SOT_SMD:SOT-143, symbol Power_Protection:PRTR5V0U2X
- added F1: MSMF010 0.01A, Fuse:Fuse_1812_4532Metric_Pad1.30x3.40mm_HandSolder, symbol Device:Polyfuse
- added J2: Conn_ST_STDC14, Connector_PinHeader_1.27mm:PinHeader_2x07_P1.27mm_Vertical_SMD, symbol Connector:Conn_ST_STDC14
- added J3: USB Type-C, Connector_USB:USB_C_Receptacle_XKB_U262-16XN-4BVC11, symbol Connector:USB_C_Receptacle_USB2.0
- added R7, R8: 5k1, Resistor_SMD:R_0805_2012Metric_Pad1.20x1.40mm_HandSolder, symbol Device:R
- added R9: 10k, Resistor_SMD:R_0805_2012Metric_Pad1.20x1.40mm_HandSolder, symbol Device:R
- added U1: STM32L412K8Tx, Package_QFP:LQFP-32_7x7mm_P0.8mm, symbol MCU_ST_STM32L4:STM32L412K8Tx
- added U7: L78L33ABUTR, Package_TO_SOT_SMD:SOT-89-3_Handsoldering, symbol Regulator_Linear:L78L33_SOT89
- added Y1: SC-32S32.768, Crystal:Crystal_SMD_EuroQuartz_EQ161-2Pin_3.2x1.5mm_HandSoldering, symbol Device:Crystal
- BT1: value 2032 Cell -> CR2032
- R2: value 10k -> 1M; LCSC Part C84376 -> C107700; Part RC0805FR-0710KL -> RC0805FR-071ML; URL https://www.lcsc.com/product-detail/Chip-Resistor-Surface-Mount_YAGEO-RC0805FR-0710KL_C84376.html -> https://www.lcsc.com/product-detail/Chip-Resistor-Surface-Mount_YAGEO-RC0805FR-071ML_C107700.html
- R6: value 100k -> 10k; LCSC Part C96346 -> C84376; Part RC0805FR-07100KL -> RC0805FR-0710KL; URL https://www.lcsc.com/product-detail/Chip-Resistor-Surface-Mount_YAGEO-RC0805FR-07100KL_C96346.html -> https://www.lcsc.com/product-detail/Chip-Resistor-Surface-Mount_YAGEO-RC0805FR-0710KL_C84376.html
Connections:
- net +3V0: now also U7.1 (OUT); no longer R2.1
- net GND: now also R2.2, C17.2, C18.2, C19.2, C20.2, J3.A1 (GND), J3.A12 (GND), J3.B1 (GND), J3.B12 (GND), R7.1, R8.1, R9.2, U1.16 (VSS), U1.32 (VSS), U7.2 (GND); no longer R6.2
- net SWDCLK: now also J2.6 (JCLK/SWCLK)
- net SWDIO: now also J2.4 (JTMS/SWDIO)
- net _RESET: now also J2.12 (~{RST}), U1.4 (NRST); no longer R2.2
- net VDDANA: now reaches C4.1, C6.1, FB1.2
- net VDDCODE: now reaches C10.1, C8.1
- net at Q1.3 (D): now also F1.1; no longer BT1.1 (+)
- net +5V: now reaches Q1.1 (G), R6.1
- net +5V: now also C20.1, D2.1 (K), D3.4 (VCC), U7.3 (IN)
- new net: C19.1, D3.1 (GND), J3.S1 (SHIELD), R2.1
- new net: J3.A5 (CC1), R7.2
- new net: D2.2 (A), J3.A4 (VBUS), J3.A9 (VBUS), J3.B4 (VBUS), J3.B9 (VBUS)
- new net: J3.B5 (CC2), R8.2
- new net: BT1.1 (+), F1.2
- new net: J2.5 (GND), J2.7 (GND)
- new net SWO: J2.8 (JTDO/SWO)
- new net USB_DM: D3.3 (I/O2), J3.A7 (D-), J3.B7 (D-)
- new net USB_DP: D3.2 (I/O1), J3.A6 (D+), J3.B6 (D+)
- new net USB_VBUS_SENSE: R6.2, R9.1
- new net XIN32: C17.1, Y1.1
- new net XOUT32: C18.1, Y1.2
- no-connect marks 18 -> 19
Other:
- note added: "D+/D- is differential pair Zdiff (differential impedance) is equal to 2 * Zodd, so a Zodd of 45 Ω gives us a Zdiff of 90 Ω"
- note added: "TODO check internal pull-up and +3V3 connection"
- note added: "TODO: USB-C connector has mounting pins. The footprint should be updated accordingly."
- note added: "TODO: check AN4879 Ann note about STM USB"
- note added: "TODO: check _RESET 100n cap"
- note added: "TODO: now it has name LSE instead of XOSC, verify 22p caps"
- moved on the sheet: D1, R1, R3, R4, R5
