File: hardware/iot-risk-logger-stm32l4.kicad_sch (KiCad schematic)
At the start: 48 parts, among them J1 USB Type-C, J5 TagConnect SWD ARM, Q1 IRLML6401, U1 ST25DV04K, U2 OPT3001DNPR, U3 SHT30-DIS, U3 W25Q64JV, U4 LIS2DW12, U5 AP2112K-3.3, U7 STM32L412, Y1 32.768

Commit message: README: update schematics
Connections:
- net GND: no longer U2.2 (ADDR)
- net VDD: now also U2.2 (ADDR)
Other:
- note added: "I2C 0x19 (0x32/0x33), ADDR(SA0)=VDD (internal pull-up)"
- note added: "I2C 0x44 (0x88/0x89), ADDR=GND"
- note added: "I2C 0x45 (0x8A/0x8B), ADDR=VDD"
- note added: "I2C: system 0x57 (0xAE/0xAF), user 0x54 (0xA6/0xA7)"
- note removed: "0x44, ADDR=L"
- note removed: "I2C 0x??, ADDR=GND"
Changed lines of the file:
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@@
   (junction (at 71.755 220.98) (diameter 0) (color 0 0 0 0)
   )
+  (junction (at 132.08 137.16) (diameter 0) (color 0 0 0 0)
+  )
   (junction (at 59.055 220.98) (diameter 0) (color 0 0 0 0)
   )
@@
     (stroke (width 0) (type default))
   )
+  (wire (pts (xy 134.62 142.24) (xy 132.08 142.24))
+    (stroke (width 0) (type default))
+  )
   (wire (pts (xy 63.5 41.91) (xy 63.5 31.75))
     (stroke (width 0) (type default))
@@
     (stroke (width 0) (type default))
   )
-  (wire (pts (xy 125.73 137.16) (xy 125.73 134.62))
+  (wire (pts (xy 132.08 137.16) (xy 132.08 134.62))
     (stroke (width 0) (type default))
   )
@@
     (stroke (width 0) (type default))
   )
+  (wire (pts (xy 132.08 142.24) (xy 132.08 137.16))
+    (stroke (width 0) (type default))
+  )
   (wire (pts (xy 64.77 135.89) (xy 62.23 135.89))
     (stroke (width 0) (type default))
@@
     (stroke (width 0) (type default))
   )
-  (wire (pts (xy 125.73 142.24) (xy 134.62 142.24))
-    (stroke (width 0) (type default))
-  )
   (bus (pts (xy 146.05 219.71) (xy 146.05 222.25))
     (stroke (width 0) (type default))
@@
     (stroke (width 0) (type default))
   )
-  (wire (pts (xy 125.73 137.16) (xy 134.62 137.16))
-    (stroke (width 0) (type default))
-  )
   (wire (pts (xy 71.755 231.14) (xy 71.755 229.87))
     (stroke (width 0) (type default))
@@
     (stroke (width 0) (type default))
   )
+  (wire (pts (xy 132.08 137.16) (xy 134.62 137.16))
+    (stroke (width 0) (type default))
+  )
   (wire (pts (xy 179.07 50.8) (xy 182.88 50.8))
     (stroke (width 0) (type default))
@@
     (stroke (width 0) (type default))
   )
-  (wire (pts (xy 125.73 158.75) (xy 125.73 142.24))
-    (stroke (width 0) (type default))
-  )
   (wire (pts (xy 191.77 50.8) (xy 191.77 48.26))
     (stroke (width 0) (type default))
@@
     (fill (type none))
   )
-  (rectangle (start 307.34 107.95) (end 400.05 173.99)
+  (rectangle (start 307.34 105.41) (end 400.05 173.99)
     (stroke (width 0) (type dash))
     (fill (type none))
@@
     (fill (type none))
   )
-  (rectangle (start 16.51 102.87) (end 107.95 168.91)
+  (rectangle (start 16.51 100.33) (end 107.95 168.91)
     (stroke (width 0) (type dash))
     (fill (type none))
@@
     (effects (font (size 2.54 2.54) (thickness 0.508) bold) (justify left bottom))
   )
-  (text "ST25DV ultra-low power: AN5733" (at 24.13 113.665 0)
+  (text "ST25DV ultra-low power: AN5733" (at 24.13 113.03 0)
     (effects (font (size 1.27 1.27)) (justify left bottom) (href "https://www.st.com/resource/en/application_note/an5733-using-st25dvi2c-series-for-ultralow-power-applications-stmicroelectronics.pdf"))
   )
@@
     (effects (font (size 2.54 2.54) (thickness 0.508) bold) (justify left bottom))
   )
-  (text "Antenna design double-layer : AN5605" (at 24.13 118.745 0)
+  (text "Antenna design double-layer : AN5605" (at 24.13 118.11 0)
     (effects (font (size 1.27 1.27)) (justify left bottom) (href "https://www.st.com/resource/en/application_note/an5605-design-of-a-1356-mhz-doublelayer-antenna-stmicroelectronics.pdf"))
   )
-  (text "FTM Data exchange: AN4910" (at 24.13 121.285 0)
+  (text "FTM Data exchange: AN4910" (at 24.13 120.65 0)
     (effects (font (size 1.27 1.27)) (justify left bottom) (href "https://www.st.com/resource/en/application_note/an4910-data-exchange-between-wired-ic-and-wireless-rf-iso-15693-using-fast-transfer-mode-supported-by-st25dvi2c-series-stmicroelectronics.pdf"))
   )
-  (text "3-AXIS ACCELEROMETER" (at 310.515 116.205 0)
+  (text "3-AXIS ACCELEROMETER" (at 311.15 113.03 0)
     (effects (font (size 2.54 2.54) (thickness 0.508) bold) (justify left bottom))
   )
@@
     (effects (font (size 1.27 1.27)) (justify left bottom))
   )
-  (text "0x44, ADDR=L" (at 231.14 168.91 0)
+  (text "I2C 0x44 (0x88/0x89), ADDR=GND" (at 214.63 116.84 0)
+    (effects (font (size 1.27 1.27)) (justify left bottom))
+  )
+  (text "I2C: system 0x57 (0xAE/0xAF), user 0x54 (0xA6/0xA7)"
+    (at 24.13 109.22 0)
     (effects (font (size 1.27 1.27)) (justify left bottom))
   )
-  (text "Antenna design: AN2972" (at 24.13 116.205 0)
+  (text "Antenna design: AN2972" (at 24.13 115.57 0)
     (effects (font (size 1.27 1.27)) (justify left bottom) (href "https://www.st.com/resource/en/application_note/an2972-how-to-design-an-antenna-for-dynamic-nfc-tags-stmicroelectronics.pdf"))
   )
@@
     (effects (font (size 2.54 2.54) (thickness 0.508) bold) (justify left bottom))
   )
+  (text "I2C 0x19 (0x32/0x33), ADDR(SA0)=VDD (internal pull-up)"
+    (at 311.15 115.57 0)
+    (effects (font (size 1.27 1.27)) (justify left bottom))
+  )
   (text "USB-C: POWER & MSD" (at 307.34 24.13 0)
     (effects (font (size 2.54 2.54) (thickness 0.508) bold) (justify left bottom))
@@
     (effects (font (size 1.27 1.27)) (justify left bottom))
   )
-  (text "I2C 0x??, ADDR=GND" (at 123.19 119.38 0)
+  (text "I2C 0x45 (0x8A/0x8B), ADDR=VDD" (at 123.19 119.38 0)
     (effects (font (size 1.27 1.27)) (justify left bottom))
   )
@@
     (effects (font (size 1.27 1.27)) (justify left bottom) (href "https://data.energizer.com/pdfs/cr2032.pdf"))
   )
-  (text "NFC\n" (at 24.13 111.125 0)
+  (text "NFC\n" (at 24.13 106.68 0)
     (effects (font (size 2.54 2.54) (thickness 0.508) bold) (justify left bottom))
   )
@@
     )
   )
-  (symbol (lib_id "power:VDD") (at 125.73 134.62 0) (unit 1)
+  (symbol (lib_id "power:VDD") (at 132.08 134.62 0) (unit 1)
     (in_bom yes) (on_board yes) (dnp no) (fields_autoplaced)
-    (property "Reference" "#PWR08" (at 125.73 138.43 0)
+    (property "Reference" "#PWR08" (at 132.08 138.43 0)
       (effects (font (size 1.27 1.27)) hide)
     )
-    (property "Value" "VDD" (at 125.73 129.54 0)
+    (property "Value" "VDD" (at 132.08 129.54 0)
       (effects (font (size 1.27 1.27)))
     )
-    (property "Footprint" "" (at 125.73 134.62 0)
+    (property "Footprint" "" (at 132.08 134.62 0)
       (effects (font (size 1.27 1.27)) hide)
     )
-    (property "Datasheet" "" (at 125.73 134.62 0)
+    (property "Datasheet" "" (at 132.08 134.62 0)
       (effects (font (size 1.27 1.27)) hide)
     )
@@
         )
       )
-    )
-  )
-  (symbol (lib_id "power:GND") (at 125.73 158.75 0) (mirror y) (unit 1)
-    (in_bom yes) (on_board yes) (dnp no) (fields_autoplaced)
-    (property "Reference" "#PWR020" (at 125.73 165.1 0)
-      (effects (font (size 1.27 1.27)) hide)
-    )
-    (property "Value" "GND" (at 125.73 163.83 0)
-      (effects (font (size 1.27 1.27)))
-    )
-    (property "Footprint" "" (at 125.73 158.75 0)
-      (effects (font (size 1.27 1.27)) hide)
-    )
-    (property "Datasheet" "" (at 125.73 158.75 0)
-      (effects (font (size 1.27 1.27)) hide)
-    )
-    (pin "1")
-    (instances
-      (project "iot-risk-logger-stm32l4"
-        (path "/a0c78d85-b3f6-4318-9ed0-83640f187f18"
-          (reference "#PWR020") (unit 1)
-        )
-      )
-      (project "iot-data-logger-nfc-samd21"
-        (path "/a430d7dc-28bf-48df-bb1e-9c942d21db4d"
-          (reference "#PWR036") (unit 1)
-        )
-      )
