File: hardware/iot-risk-logger-stm32l4.kicad_sch (KiCad schematic)
At the start: 58 parts, among them J1 USB Type-C, J2 TagConnect SWD ARM, Q1 AO3407, U1 ST25DV04K, U2 OPT3001DNPR, U3 SHT30-DIS, U4 LIS2DW12, U5 AP2112K-3.3, U6 W25Q64JV, U7 SiP32431DR3, U8 STM32L433CBTx, Y1 32.768

Commit message: :construction: wip(SCH/PCB) update schematics, pcb and generate fabrications
Parts:
- removed C1, C20, C5, C7: 10u, Capacitor_SMD:C_0805_2012Metric_Pad1.18x1.45mm_HandSolder, symbol Device:C
- removed FB1: 330, Resistor_SMD:R_0805_2012Metric_Pad1.20x1.40mm_HandSolder, symbol Device:FerriteBead_Small
- removed R3: 1k, Resistor_SMD:R_0805_2012Metric_Pad1.20x1.40mm_HandSolder, symbol Device:R
- removed R5: 5k1, Resistor_SMD:R_0603_1608Metric_Pad0.98x0.95mm_HandSolder, symbol Device:R
- added C15, C3: 10u, Capacitor_SMD:C_0805_2012Metric_Pad1.18x1.45mm_HandSolder, symbol Device:C
- added FB1: 330, Inductor_SMD:L_0805_2012Metric_Pad1.15x1.40mm_HandSolder, symbol Device:FerriteBead
- added R11, R8: 2k2, Resistor_SMD:R_0603_1608Metric_Pad0.98x0.95mm_HandSolder, symbol Device:R
- C12: value 100u -> 100n; footprint Capacitor_SMD:C_0805_2012Metric_Pad1.18x1.45mm_HandSolder -> Capacitor_SMD:C_0603_1608Metric_Pad1.08x0.95mm_HandSolder; LCSC Part # (none) -> C1591; LCSC URL (none) -> https://www.lcsc.com/product-detail/Multilayer-Ceramic-Capa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; Manufacturer Samsung Electro-Mechanics -> Samsung Electro-Mechanics; Mfr. Part # (none) -> CL10B104KB8NNNC
- Q1: LCSC Part # (none) -> C2938376; LCSC URL (none) -> https://www.lcsc.com/product-detail/C2938376.html; Manufacturer (none) -> GOODWORK; Mfr. Part # (none) -> AO3407
- R10, R12: value 5k1 -> 2k2; LCSC Part # C14677 -> C113303; LCSC URL https://www.lcsc.com/product-detail/Chip-Resistor-Surface-M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 -> https://www.lcsc.com/product-detail/C113303.html; Mfr. Part # RC0603JR-075K1L -> RC0603JR-072K2L
- R3: renamed from R8; LCSC Part # C137678 -> C141684; LCSC URL https://www.lcsc.com/product-detail/Chip-Resistor-Surface-M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 -> https://www.lcsc.com/product-detail/C141684.html?s_z=n_820k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; Mfr. Part # RC0603FR-0782KL -> RC0603FR-07820KL
- R4: renamed from R9; LCSC Part # C126359 -> C114618; LCSC URL https://www.lcsc.com/product-detail/Chip-Resistor-Surface-M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 -> https://www.lcsc.com/product-detail/C114618.html?s_z=n_RC06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; Mfr. Part # RC0603FR-0733KL -> RC0603FR-07330KL
- R9: renamed from R4; value 5k1 -> 2k2; LCSC Part # C14677 -> C113303; LCSC URL https://www.lcsc.com/product-detail/Chip-Resistor-Surface-M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 -> https://www.lcsc.com/product-detail/C113303.html; Mfr. Part # RC0603JR-075K1L -> RC0603JR-072K2L
- TP1: renamed from TP3; value TP: GND -> GND; footprint TestPoint:TestPoint_THTPad_D1.5mm_Drill0.7mm -> TestPoint:TestPoint_Pad_D1.5mm
- TP2: renamed from TP4; footprint TestPoint:TestPoint_THTPad_D1.5mm_Drill0.7mm -> TestPoint:TestPoint_Pad_D1.5mm
- TP3: renamed from TP1; footprint TestPoint:TestPoint_THTPad_D1.5mm_Drill0.7mm -> TestPoint:TestPoint_Pad_D1.5mm
- TP4: renamed from TP2; footprint TestPoint:TestPoint_THTPad_D1.5mm_Drill0.7mm -> TestPoint:TestPoint_Pad_D1.5mm
- TP5, TP6: footprint TestPoint:TestPoint_THTPad_D1.5mm_Drill0.7mm -> TestPoint:TestPoint_Pad_D1.5mm
- U3: renamed from U2; footprint Personal:SON65P200X200X65-7N -> personal:SON65P200X200X65-7N
- U4: renamed from U3; value SHT30-DIS -> SHT31-DIS; LCSC Part # C2687423 -> C80862; LCSC URL https://www.lcsc.com/product-detail/Temperature-and-Humidit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 -> https://item.szlcsc.com/82012.html; Mfr. Part # SHT30-DIS-B10KS -> SHT31-DIS-B2.5kS
- U6: value W25Q64JV -> AT25SF161B; footprint Package_SO:SOIC-8_5.23x5.23mm_P1.27mm -> Package_SO:SOIC-8_3.9x4.9mm_P1.27mm; LCSC Part # C83140 -> C5555633; LCSC URL https://www.lcsc.com/product-detail/NOR-FLASH_Winbond-Elec-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 -> https://www.lcsc.com/product-detail/C5555633.html; Manufacturer Winbond -> RENESAS; Mfr. Part # W25Q64JVSSIQ -> AT25SF161B-SSHD-B
- U7: renamed from U8; value STM32L433CBTx -> STM32L433CCT6; LCSC Part # (none) -> C110061; LCSC URL (none) -> https://www.lcsc.com/product-detail/C110061.html; Manufacturer (none) -> ST; Mfr. Part # (none) -> STM32L433CCT6
- U8: renamed from U7; LCSC Part # (none) -> C141606; LCSC URL (none) -> https://www.lcsc.com/product-detail/C141606.html; Manufacturer (none) -> VISHAY; Mfr. Part # (none) -> SIP32431DR3-T1GE3
- renumbered C8 to C1, C3 to C10, C4 to C11, C6 to C13, C9 to C14, C18 to C16, C16 to C18, C15 to C19, C21 to C2, C14 to C4, C13 to C5, C11 to C6, C19 to C7, C10 to C8, C2 to C9, D4 to D2, D2 to D4, R7 to R5, R11 to R6, R6 to R7, U5 to U1, U1 to U2, U4 to U5
Connections:
- net +3V0: now also FB1.1
- net +LED: now also R8.2
- net GND: now also C15.2, C3.2
- net I2C1_SCL_SENS: now also R10.2
- net I2C2_SDA_NFC: now also R11.2; no longer R10.2
- net VDD: now also C12.1, R10.1, U7.1 (VBAT), U7.24 (VDD), U7.36 (VDDUSB), U7.48 (VDD), U7.9 (VDDA), C3.1, FB1.2, R8.1
- net VDD_MEMORY: now also C15.1; no longer C12.1
- net VDD_NFC: now also R11.1; no longer R10.1
- net USB_DM_N renamed USB_DN
- net USB_DP_P renamed USB_DP
Other:
- note added: "2.5V - 3.6V: allows to drain battery effeciently"
- note added: "I = 0.45mA"
- note added: "QSPI NOR FLASH 2MB"
- note removed: "I = 1mA"
- note removed: "QSPI NOR FLASH 8MB"
- note removed: "TODO: USB_SENSE on WKUP"
- note removed: "TODO: can CS QSPI_NCS_N be connected to GND? TODO: R6 necessity?"
- note removed: "TODO: move LED accordingly"
- note removed: "W25Q works down to 2V7, better to replace by 2V4 memory"
- moved on the sheet: AE1, C10, C11, C13, C2, C4, C5, C6, C7, C9, D4, R6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
