File: hardware/iot-risk-logger-stm32l4.kicad_sch (KiCad schematic)
At the start: 48 parts, among them J1 USB Type-C, J5 TagConnect SWD ARM, Q1 IRLML6401, U1 ST25DV04K, U2 OPT3001DNPR, U3 SHT30-DIS, U3 W25Q64JV, U4 LIS2DW12, U5 AP2112K-3.3, U7 STM32L412, Y1 32.768

Commit message: PCB: add colours and board extraction cutout
Other:
- moved on the sheet: AE1, C1, C10, C11, C13, C14, C2, C3, C4, C5, C6, C7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

Commit message: :construction: wip(SCH/PCB) draft schematics with STM32L433 and evolved power rails
Parts:
- removed R19: 10k, Resistor_SMD:R_0603_1608Metric_Pad0.98x0.95mm_HandSolder, symbol Device:R
- removed U7: STM32L412, Package_QFP:LQFP-32_7x7mm_P0.8mm, symbol MCU_ST_STM32L4:STM32L412K8Tx
- added C12: 100u, Capacitor_SMD:C_0805_2012Metric_Pad1.18x1.45mm_HandSolder, symbol Device:C
- added C19: 100n, Capacitor_SMD:C_0603_1608Metric_Pad1.08x0.95mm_HandSolder, symbol Device:C
- added C20, C21: 10u, Capacitor_SMD:C_0805_2012Metric_Pad1.18x1.45mm_HandSolder, symbol Device:C
- added D4: BAT60A, Diode_SMD:D_SOD-323_HandSoldering, symbol Diode:BAT60A
- added R10, R12: 5k1, Resistor_SMD:R_0603_1608Metric_Pad0.98x0.95mm_HandSolder, symbol Device:R
- added R11: 10k, Resistor_SMD:R_0603_1608Metric_Pad0.98x0.95mm_HandSolder, symbol Device:R
- added TP5: TP: I2C2_SDA_NFC, TestPoint:TestPoint_THTPad_D1.5mm_Drill0.7mm, symbol Connector:TestPoint_Probe
- added TP6: TP: I2C2_SCL_NFC, TestPoint:TestPoint_THTPad_D1.5mm_Drill0.7mm, symbol Connector:TestPoint_Probe
- added U7: SiP32431DR3, Package_TO_SOT_SMD:SOT-363_SC-70-6, symbol Power_Management:SiP32431DR3
- added U8: STM32L433CBTx, Package_QFP:LQFP-48_7x7mm_P0.5mm, symbol MCU_ST_STM32L4:STM32L433CBTx
- Q1: value IRLML6401 -> AO3407; LCSC Part # C3034 -> (none); LCSC URL https://www.lcsc.com/product-detail/MOSFETs_Infineon-Techno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 -> (none); Manufacturer Infineon -> (none); Mfr. Part # IRLML6401TRPBF -> (none)
- R8: value 82k -> 820k
- R9: value 33k -> 330k
- TP1: value TP: SDA -> TP: I2C1_SDA_SENS
- TP2: value TP: SCL -> TP: I2C1_SCL_SENS
- TP4: value TP: NFC_INT -> TP: NFC_INT_WKUP
- renumbered C10 to C16, C10 to C17, D5 to D2, J5 to J2, R15 to R3, R19 to R6, U3 to U6
Connections:
- net +3V0: now also C21.1, D4.1 (K); no longer U5.5 (VOUT)
- net GND: now also C12.2, C19.2, C20.2, C21.2, U7.2 (GND), U7.5 (GND), U8.23 (VSS), U8.35 (VSS), U8.44 (PH3), U8.47 (VSS), U8.8 (VSSA)
- net IMU_INT1: now also U8.42 (PB6)
- net IMU_INT2: now also U8.43 (PB7)
- net QSPI_CLK: now also U8.13 (PA3)
- net QSPI_IO0: now also U8.19 (PB1)
- net QSPI_IO1: now also U8.18 (PB0)
- net QSPI_IO2: now also U8.17 (PA7)
- net QSPI_IO3: now also U8.16 (PA6)
- net SWDIO: now also U8.34 (PA13)
- net SWO: now also U8.39 (PB3)
- net TEMP_INT: now also U8.41 (PB5)
- net VDD: now also C19.1, C20.1, R11.2, U7.4 (IN); no longer C1.1, C2.1, C9.1, R6.2, U1.8 (VCC), U6.8 (VCC)
- net LSE_IN renamed RCC_OSC32_IN
- net RCC_OSC32_IN: now also U8.3 (PC14)
- net LSE_OUT renamed RCC_OSC32_OUT
- net RCC_OSC32_OUT: now also U8.4 (PC15)
- net SCL renamed I2C1_SCL_SENS
- net I2C1_SCL_SENS: now also U8.30 (PA9); no longer U1.6 (SCL)
- net SDA renamed I2C1_SDA_SENS
- net I2C1_SDA_SENS: now also U8.31 (PA10); no longer U1.5 (SDA)
- net SWDCLK renamed SWCLK
- net SWCLK: now also U8.37 (PA14)
- net USB_N renamed USB_DM_N
- net USB_DM_N: now also U8.32 (PA11)
- net USB_P renamed USB_DP_P
- net USB_DP_P: now also U8.33 (PA12)
- net USB_VBUS_SENSE renamed USB_VBUS_SENSE_WKUP2
- net USB_VBUS_SENSE_WKUP2: now also U8.2 (PC13)
- net _LED renamed LED_N
- net LED_N: now also U8.38 (PA15)
- net _LIGHT_INT renamed LIGHT_INT_N
- net LIGHT_INT_N: now also U8.45 (PB8)
- net _NFC_INT renamed NFC_INT_WKUP
- net NFC_INT_WKUP: now also R11.1, U8.10 (PA0)
- net _QSPI_NCS renamed QSPI_NCS_N
- net QSPI_NCS_N: now also U8.12 (PA2)
- net _RESET renamed RESET_N
- net RESET_N: now also U8.7 (NRST)
- net _TEMP_RESET renamed TEMPRESET_N
- net TEMPRESET_N: now also U8.40 (PB4)
- new net: D4.2 (A), U5.5 (VOUT)
- new net I2C2_SCL_NFC: R12.2, TP6.1, U1.6 (SCL), U8.21 (PB10)
- new net I2C2_SDA_NFC: R10.2, TP5.1, U1.5 (SDA), U8.22 (PB11)
- new net MEMORY_EN: U7.3 (ON), U8.14 (PA4)
- new net VDD_MEMORY: C12.1, C9.1, R6.2, U6.8 (VCC), U7.1 (OUT)
- new net VDD_NFC: C1.1, C2.1, R10.1, R12.1, U1.8 (VCC), U8.20 (PB2)
- no-connect marks 8 -> 16
Other:
- note added: "LOW-PASS FILTER & MCU CAPS"
- note added: "Memory load switch"
- note added: "TODO: USB_SENSE on WKUP"
- note added: "TODO: can CS QSPI_NCS_N be connected to GND? TODO: R6 necessity?"
- note added: "TODO: move LED accordingly"
- note removed: "LOW-PASS FILTER"
- note removed: "MCU CAPS"
- moved on the sheet: AE1, C1, C11, C13, C14, C16, C17, C2, C3, C4, C5, C6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

Commit message: :construction: wip(SCH/PCB) update schematics, pcb and generate fabrications
Parts:
- removed C1, C20, C5, C7: 10u, Capacitor_SMD:C_0805_2012Metric_Pad1.18x1.45mm_HandSolder, symbol Device:C
- removed FB1: 330, Resistor_SMD:R_0805_2012Metric_Pad1.20x1.40mm_HandSolder, symbol Device:FerriteBead_Small
- removed R3: 1k, Resistor_SMD:R_0805_2012Metric_Pad1.20x1.40mm_HandSolder, symbol Device:R
- removed R5: 5k1, Resistor_SMD:R_0603_1608Metric_Pad0.98x0.95mm_HandSolder, symbol Device:R
- added C15, C3: 10u, Capacitor_SMD:C_0805_2012Metric_Pad1.18x1.45mm_HandSolder, symbol Device:C
- added FB1: 330, Inductor_SMD:L_0805_2012Metric_Pad1.15x1.40mm_HandSolder, symbol Device:FerriteBead
- added R11, R8: 2k2, Resistor_SMD:R_0603_1608Metric_Pad0.98x0.95mm_HandSolder, symbol Device:R
- C12: value 100u -> 100n; footprint Capacitor_SMD:C_0805_2012Metric_Pad1.18x1.45mm_HandSolder -> Capacitor_SMD:C_0603_1608Metric_Pad1.08x0.95mm_HandSolder; LCSC Part # (none) -> C1591; LCSC URL (none) -> https://www.lcsc.com/product-detail/Multilayer-Ceramic-Capa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; Manufacturer Samsung Electro-Mechanics -> Samsung Electro-Mechanics; Mfr. Part # (none) -> CL10B104KB8NNNC
- Q1: LCSC Part # (none) -> C2938367; LCSC URL (none) -> https://www.lcsc.com/product-detail/C2938367.html?s_z=n_AO3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; Manufacturer (none) -> GOODWORK; Mfr. Part # (none) -> AO3400
- R10, R12: value 5k1 -> 2k2; LCSC Part # C14677 -> C113303; LCSC URL https://www.lcsc.com/product-detail/Chip-Resistor-Surface-M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 -> https://www.lcsc.com/product-detail/C113303.html; Mfr. Part # RC0603JR-075K1L -> RC0603JR-072K2L
- R3: renamed from R8; LCSC Part # C137678 -> C141684; LCSC URL https://www.lcsc.com/product-detail/Chip-Resistor-Surface-M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 -> https://www.lcsc.com/product-detail/C141684.html?s_z=n_820k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; Mfr. Part # RC0603FR-0782KL -> RC0603FR-07820KL
- R4: renamed from R9; LCSC Part # C126359 -> C114618; LCSC URL https://www.lcsc.com/product-detail/Chip-Resistor-Surface-M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 -> https://www.lcsc.com/product-detail/C114618.html?s_z=n_RC06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; Mfr. Part # RC0603FR-0733KL -> RC0603FR-07330KL
- R9: renamed from R4; value 5k1 -> 2k2; LCSC Part # C14677 -> C113303; LCSC URL https://www.lcsc.com/product-detail/Chip-Resistor-Surface-M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 -> https://www.lcsc.com/product-detail/C113303.html; Mfr. Part # RC0603JR-075K1L -> RC0603JR-072K2L
- TP1: renamed from TP3; value TP: GND -> GND; footprint TestPoint:TestPoint_THTPad_D1.5mm_Drill0.7mm -> TestPoint:TestPoint_Pad_D1.5mm
- TP2: renamed from TP4; footprint TestPoint:TestPoint_THTPad_D1.5mm_Drill0.7mm -> TestPoint:TestPoint_Pad_D1.5mm
- TP3: renamed from TP1; footprint TestPoint:TestPoint_THTPad_D1.5mm_Drill0.7mm -> TestPoint:TestPoint_Pad_D1.5mm
- TP4: renamed from TP2; footprint TestPoint:TestPoint_THTPad_D1.5mm_Drill0.7mm -> TestPoint:TestPoint_Pad_D1.5mm
- TP5, TP6: footprint TestPoint:TestPoint_THTPad_D1.5mm_Drill0.7mm -> TestPoint:TestPoint_Pad_D1.5mm
- U3: renamed from U2; footprint Personal:SON65P200X200X65-7N -> personal:SON65P200X200X65-7N
- U4: renamed from U3; value SHT30-DIS -> SHT31-DIS; LCSC Part # C2687423 -> C80862; LCSC URL https://www.lcsc.com/product-detail/Temperature-and-Humidit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 -> https://item.szlcsc.com/82012.html; Mfr. Part # SHT30-DIS-B10KS -> SHT31-DIS-B2.5kS
- U6: value W25Q64JV -> AT25SF161B; footprint Package_SO:SOIC-8_5.23x5.23mm_P1.27mm -> Package_SO:SOIC-8_3.9x4.9mm_P1.27mm; LCSC Part # C83140 -> C5555633; LCSC URL https://www.lcsc.com/product-detail/NOR-FLASH_Winbond-Elec-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 -> https://www.lcsc.com/product-detail/C5555633.html; Manufacturer Winbond -> RENESAS; Mfr. Part # W25Q64JVSSIQ -> AT25SF161B-SSHD-B
- U7: renamed from U8; value STM32L433CBTx -> STM32L433CCT6; LCSC Part # (none) -> C110061; LCSC URL (none) -> https://www.lcsc.com/product-detail/C110061.html; Manufacturer (none) -> ST; Mfr. Part # (none) -> STM32L433CCT6
- U8: renamed from U7; LCSC Part # (none) -> C141606; LCSC URL (none) -> https://www.lcsc.com/product-detail/C141606.html; Manufacturer (none) -> VISHAY; Mfr. Part # (none) -> SIP32431DR3-T1GE3
- renumbered C8 to C1, C3 to C10, C4 to C11, C6 to C13, C9 to C14, C18 to C16, C16 to C18, C15 to C19, C21 to C2, C14 to C4, C13 to C5, C11 to C6, C19 to C7, C10 to C8, C2 to C9, D4 to D2, D2 to D4, R7 to R5, R11 to R6, R6 to R7, U5 to U1, U1 to U2, U4 to U5
Connections:
- net +3V0: now also FB1.1
- net +LED: now also R8.2
- net GND: now also C15.2, C3.2
- net I2C1_SCL_SENS: now also R10.2
- net I2C2_SDA_NFC: now also R11.2; no longer R10.2
- net VDD: now also C12.1, R10.1, U7.1 (VBAT), U7.24 (VDD), U7.36 (VDDUSB), U7.48 (VDD), U7.9 (VDDA), C3.1, FB1.2, R8.1
- net VDD_MEMORY: now also C15.1; no longer C12.1
- net VDD_NFC: now also R11.1; no longer R10.1
- net USB_DM_N renamed USB_DN
- net USB_DP_P renamed USB_DP
Other:
- note added: "2.5V - 3.6V: allows to drain battery effeciently"
- note added: "I = 0.45mA"
- note added: "QSPI NOR FLASH 2MB"
- note removed: "I = 1mA"
- note removed: "QSPI NOR FLASH 8MB"
- note removed: "TODO: USB_SENSE on WKUP"
- note removed: "TODO: can CS QSPI_NCS_N be connected to GND? TODO: R6 necessity?"
- note removed: "W25Q works down to 2V7, better to replace by 2V4 memory"
- moved on the sheet: AE1, C10, C11, C13, C2, C4, C5, C6, C7, C9, D4, R6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
