File: hardware/iot-risk-logger-stm32l4.kicad_pcb (KiCad board)
At the start: 2 copper layers, 55 x 45 mm, 52 parts, among them J1 USB Type-C, J2 TagConnect SWD ARM, Q1 IRLML6401, U1 ST25DV04K, U2 OPT3001DNPR, U3 SHT30-DIS, U4 LIS2DW12, U5 AP2112K-3.3, U6 W25Q64JV, U7 STM32L412, Y1 32.768

Commit message: :construction: wip(SCH/PCB) draft schematics with STM32L433 and evolved power rails
Parts:
- added C12: 100u, Capacitor_SMD:C_0805_2012Metric_Pad1.18x1.45mm_HandSolder, F.Cu at (91.4, 26.9)
- added C19: 100n, Capacitor_SMD:C_0603_1608Metric_Pad1.08x0.95mm_HandSolder, F.Cu at (101.1, 35.0)
- added C20: 10u, Capacitor_SMD:C_0805_2012Metric_Pad1.18x1.45mm_HandSolder, F.Cu at (91.4, 29.9)
- added C21: 10u, Capacitor_SMD:C_0805_2012Metric_Pad1.18x1.45mm_HandSolder, F.Cu at (91.4, 32.9)
- added C7: 10u, Capacitor_SMD:C_0805_2012Metric_Pad1.18x1.45mm_HandSolder, F.Cu at (91.4, 23.9)
- added D4: BAT60A, Diode_SMD:D_SOD-323_HandSoldering, F.Cu at (96.4, 35.2)
- added R11: 10k, Resistor_SMD:R_0603_1608Metric_Pad0.98x0.95mm_HandSolder, F.Cu at (101.1, 37.5)
- added U7: SiP32431DR3, Package_TO_SOT_SMD:SOT-363_SC-70-6, F.Cu at (91.1, 36.4)
- added U8: STM32L433CBTx, Package_QFP:LQFP-48_7x7mm_P0.5mm, F.Cu at (99.5, 28.1)
- Q1: value IRLML6401 -> AO3407
- R8: value 82k -> 820k
- R9: value 33k -> 330k
- TP1: value TP: SDA -> TP: I2C1_SDA_SENS
- TP2: value TP: SCL -> TP: I2C1_SCL_SENS
- TP4: value TP: NFC_INT -> TP: NFC_INT_WKUP
Connections:
- C1 pad 1: VDD -> VDD_NFC
- C15 pad 1: _RESET -> RESET_N
- C16 pad 1: /LSE_OUT -> /RCC_OSC32_OUT
- C17 pad 1: /LSE_IN -> /RCC_OSC32_IN
- C2 pad 1: VDD -> VDD_NFC
- C9 pad 1: VDD -> /VDD_MEMORY
- D2 pad 1: _LED -> LED_N
- D3 pad 2: USB_P -> USB_DP_P
- D3 pad 3: USB_N -> USB_DM_N
- J1 pad A6: USB_P -> USB_DP_P
- J1 pad A7: USB_N -> USB_DM_N
- J1 pad B6: USB_P -> USB_DP_P
- J1 pad B7: USB_N -> USB_DM_N
- J1 pad s1: /GND_SHIELD -> (no net)
- J2 pad 10: _RESET -> RESET_N
- J2 pad 4: SWDCLK -> SWCLK
- R4 pad 2: SDA -> I2C1_SDA_SENS
- R5 pad 2: SCL -> I2C1_SCL_SENS
- R6 pad 1: /_QSPI_NCS -> /QSPI_NCS_N
- R6 pad 2: VDD -> /VDD_MEMORY
- R8 pad 2: USB_VBUS_SENSE -> USB_VBUS_SENSE_WKUP2
- R9 pad 1: USB_VBUS_SENSE -> USB_VBUS_SENSE_WKUP2
- TP1 pad 1: SDA -> I2C1_SDA_SENS
- TP2 pad 1: SCL -> I2C1_SCL_SENS
- TP4 pad 1: _NFC_INT -> NFC_INT_WKUP
- U1 pad 5: SDA -> I2C2_SDA_NFC
- U1 pad 6: SCL -> I2C2_SCL_NFC
- U1 pad 7: _NFC_INT -> NFC_INT_WKUP
- U1 pad 8: VDD -> VDD_NFC
- U2 pad 4: SCL -> I2C1_SCL_SENS
- U2 pad 5: _LIGHT_INT -> LIGHT_INT_N
- U2 pad 6: SDA -> I2C1_SDA_SENS
- U3 pad 1: SDA -> I2C1_SDA_SENS
- U3 pad 4: SCL -> I2C1_SCL_SENS
- U3 pad 6: _TEMP_RESET -> TEMPRESET_N
- U4 pad 1: SCL -> I2C1_SCL_SENS
- U4 pad 4: SDA -> I2C1_SDA_SENS
- U5 pad 5: +3V0 -> Net-(D4-A)
- U6 pad 1: /_QSPI_NCS -> /QSPI_NCS_N
- U6 pad 8: VDD -> /VDD_MEMORY
- Y1 pad 1: /LSE_IN -> /RCC_OSC32_IN
- Y1 pad 2: /LSE_OUT -> /RCC_OSC32_OUT
Routing:
- net SDA: vias 3 -> 2
- net I2C1_SDA_SENS: vias 0 -> 1

Commit message: :construction: wip(SCH/PCB) update schematics, pcb and generate fabrications
Parts:
- removed the C13 at (58.2, 39.4)
- removed the C14 at (67.6, 48.9)
- removed C21: 10u, Capacitor_SMD:C_0805_2012Metric_Pad1.18x1.45mm_HandSolder
- removed the C3 at (62.9, 31.5)
- removed the C7 at (69.2, 57.5)
- removed the C8 at (70.2, 62.4)
- removed the R6 at (51.4, 59.4)
- removed the R7 at (73.3, 49.2)
- removed the R9 at (71.5, 53.9)
- removed the U7 at (63.1, 43.9)
- added C12: 100n, Capacitor_SMD:C_0603_1608Metric_Pad1.08x0.95mm_HandSolder, F.Cu at (59.5, 41.7)
- added C15: 10u, Capacitor_SMD:C_0805_2012Metric_Pad1.18x1.45mm_HandSolder, F.Cu at (50.5, 43.1)
- added C5: 100n, Capacitor_SMD:C_0603_1608Metric_Pad1.08x0.95mm_HandSolder, F.Cu at (61.8, 34.0)
- added R1: 5k1, Resistor_SMD:R_0603_1608Metric_Pad0.98x0.95mm_HandSolder, F.Cu at (81.7, 41.1)
- added R11: 2k2, Resistor_SMD:R_0603_1608Metric_Pad0.98x0.95mm_HandSolder, F.Cu at (53.6, 38.7)
- added R4: 330k, Resistor_SMD:R_0603_1608Metric_Pad0.98x0.95mm_HandSolder, F.Cu at (76.5, 51.9)
- added R5: 1M, Resistor_SMD:R_0603_1608Metric_Pad0.98x0.95mm_HandSolder, F.Cu at (76.4, 50.4)
- added TP3: TP: I2C1_SDA_SENS, TestPoint:TestPoint_Pad_D1.5mm, F.Cu at (76.7, 27.8)
- added TP4: TP: I2C1_SCL_SENS, TestPoint:TestPoint_Pad_D1.5mm, F.Cu at (76.7, 30.4)
- C1: renamed from C19; value 100n -> 10u; footprint Capacitor_SMD:C_0603_1608Metric_Pad1.08x0.95mm_HandSolder -> Capacitor_SMD:C_0805_2012Metric_Pad1.18x1.45mm_HandSolder
- C10: renamed from C5; value 10u -> 100n; footprint Capacitor_SMD:C_0805_2012Metric_Pad1.18x1.45mm_HandSolder -> Capacitor_SMD:C_0603_1608Metric_Pad1.08x0.95mm_HandSolder
- C16: renamed from C12; value 100u -> 100n; footprint Capacitor_SMD:C_0805_2012Metric_Pad1.18x1.45mm_HandSolder -> Capacitor_SMD:C_0603_1608Metric_Pad1.08x0.95mm_HandSolder
- C17: renamed from C9; value 100n -> 22p; footprint Capacitor_SMD:C_0603_1608Metric_Pad1.08x0.95mm_HandSolder -> Capacitor_SMD:C_0603_1608Metric
- C2: renamed from C10; value 4n7 -> 10u; footprint Capacitor_SMD:C_0603_1608Metric_Pad1.08x0.95mm_HandSolder -> Capacitor_SMD:C_0805_2012Metric_Pad1.18x1.45mm_HandSolder
- C4: renamed from C20; value 10u -> 100n; footprint Capacitor_SMD:C_0805_2012Metric_Pad1.18x1.45mm_HandSolder -> Capacitor_SMD:C_0603_1608Metric_Pad1.08x0.95mm_HandSolder
- C7: renamed from C17; value 22p -> 100n; footprint Capacitor_SMD:C_0603_1608Metric -> Capacitor_SMD:C_0603_1608Metric_Pad1.08x0.95mm_HandSolder
- C8: renamed from C18; value 100n -> 4n7
- C9: renamed from C7; value 10u -> 100n; footprint Capacitor_SMD:C_0805_2012Metric_Pad1.18x1.45mm_HandSolder -> Capacitor_SMD:C_0603_1608Metric_Pad1.08x0.95mm_HandSolder
- D1: renamed from D2; value LED -> BAT60A; footprint LED_SMD:LED_0805_2012Metric_Pad1.15x1.40mm_HandSolder -> Diode_SMD:D_SOD-323_HandSoldering
- D2: renamed from D3; value PRTR5V0U2X -> BAT60A; footprint Package_TO_SOT_SMD:SOT-143 -> Diode_SMD:D_SOD-323_HandSoldering
- D3: renamed from D1; value BAT60A -> PRTR5V0U2X; footprint Diode_SMD:D_SOD-323_HandSoldering -> Package_TO_SOT_SMD:SOT-143
- D4: value BAT60A -> LED; footprint Diode_SMD:D_SOD-323_HandSoldering -> LED_SMD:LED_0805_2012Metric_Pad1.15x1.40mm_HandSolder
- FB1: footprint Resistor_SMD:R_0805_2012Metric_Pad1.20x1.40mm_HandSolder -> Inductor_SMD:L_0805_2012Metric_Pad1.15x1.40mm_HandSolder
- J1: renamed from J2; value TagConnect SWD ARM -> USB Type-C; footprint Connector:Tag-Connect_TC2050-IDC-NL_2x05_P1.27mm_Vertical_with_bottom_clip -> Connector_USB:USB_C_Receptacle_XKB_U262-16XN-4BVC11; moved to B.Cu
- J2: renamed from J1; value USB Type-C -> TagConnect SWD ARM; footprint Connector_USB:USB_C_Receptacle_XKB_U262-16XN-4BVC11 -> Connector:Tag-Connect_TC2050-IDC-NL_2x05_P1.27mm_Vertical_with_bottom_clip; moved to F.Cu
- R10: value 10k -> 2k2
- R12: renamed from R8; value 820k -> 2k2
- R2: renamed from R11; value 10k -> 5k1
- R3: renamed from R5; value 5k1 -> 820k
- R6: renamed from R2; value 5k1 -> 10k
- R7: renamed from R4; value 5k1 -> 10k
- R8: renamed from R3; value 1k -> 2k2; footprint Resistor_SMD:R_0805_2012Metric_Pad1.20x1.40mm_HandSolder -> Resistor_SMD:R_0603_1608Metric_Pad0.98x0.95mm_HandSolder
- R9: renamed from R1; value 5k1 -> 2k2
- TP1: renamed from TP4; value TP: NFC_INT_WKUP -> GND; footprint TestPoint:TestPoint_THTPad_D1.5mm_Drill0.7mm -> TestPoint:TestPoint_Pad_D1.5mm
- TP2: value TP: I2C1_SCL_SENS -> TP: NFC_INT_WKUP; footprint TestPoint:TestPoint_THTPad_D1.5mm_Drill0.7mm -> TestPoint:TestPoint_Pad_D1.5mm
- TP5: renamed from TP1; value TP: I2C1_SDA_SENS -> TP: I2C2_SDA_NFC; footprint TestPoint:TestPoint_THTPad_D1.5mm_Drill0.7mm -> TestPoint:TestPoint_Pad_D1.5mm
- TP6: renamed from TP3; value TP: GND -> TP: I2C2_SCL_NFC; footprint TestPoint:TestPoint_THTPad_D1.5mm_Drill0.7mm -> TestPoint:TestPoint_Pad_D1.5mm
- U1: renamed from U6; value W25Q64JV -> AP2112K-3.3; footprint Package_SO:SOIC-8_5.23x5.23mm_P1.27mm -> Package_TO_SOT_SMD:SOT-23-5
- U2: renamed from U4; value LIS2DW12 -> ST25DV04K; footprint Package_LGA:LGA-12_2x2mm_P0.5mm -> Package_SO:TSSOP-8_4.4x3mm_P0.65mm
- U3: renamed from U1; value ST25DV04K -> OPT3001DNPR; footprint Package_SO:TSSOP-8_4.4x3mm_P0.65mm -> personal:SON65P200X200X65-7N
- U4: renamed from U3; value SHT30-DIS -> SHT31-DIS
- U5: renamed from U2; value OPT3001DNPR -> LIS2DW12; footprint Personal:SON65P200X200X65-7N -> Package_LGA:LGA-12_2x2mm_P0.5mm
- U6: renamed from U7; value SiP32431DR3 -> AT25SF161B; footprint Package_TO_SOT_SMD:SOT-363_SC-70-6 -> Package_SO:SOIC-8_3.9x4.9mm_P1.27mm
- U7: renamed from U5; value AP2112K-3.3 -> STM32L433CCT6; footprint Package_TO_SOT_SMD:SOT-23-5 -> Package_QFP:LQFP-48_7x7mm_P0.5mm
- U8: value STM32L433CBTx -> SiP32431DR3; footprint Package_QFP:LQFP-48_7x7mm_P0.5mm -> Package_TO_SOT_SMD:SOT-363_SC-70-6
- moved U8 48.8 mm to (53.0, 42.8), turned to 90 degrees
- moved U6 39.1 mm to (54.1, 48.9), turned to 90 degrees
- moved C9 38.8 mm to (53.1, 30.0), turned to 90 degrees
- moved D4 37.2 mm to (60.5, 25.5), turned to -90 degrees
- moved R3 31.1 mm to (76.4, 53.5), turned to 180 degrees
- moved TP1 29.8 mm to (66.0, 55.2)
- moved R6 27.8 mm to (53.1, 26.7)
- moved R12 27.6 mm to (53.6, 36.2)
- moved TP5 26.6 mm to (50.7, 38.7)
- moved C1 26.5 mm to (80.8, 51.9), turned to 180 degrees
- moved U1 25.6 mm to (80.6, 56.0), turned to -90 degrees
- moved TP6 24.6 mm to (50.7, 36.2)
- moved C19 24.2 mm to (77.9, 37.3), turned to 0 degrees
- moved D1 23.7 mm to (80.8, 49.9), turned to 180 degrees
- moved U7 23.3 mm to (65.8, 39.5), turned to 0 degrees
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- renumbered C6 to C11, C2 to C13, C4 to C14, C16 to C18, C11 to C19, C1 to C3, C15 to C6, REF99 to REF1, REF98 to REF2, REF97 to REF3
Connections:
- AE1 pad 1: Net-(U1-AC1) -> Net-(U2-AC1)
- AE1 pad 2: Net-(U1-AC0) -> Net-(U2-AC0)
- C1 pad 1: VDD -> +5V
- C13 pad 1: VDD_NFC -> VDD
- C14 pad 1: VDD -> /VDD_MEMORY
- C16 pad 1: /VDD_MEMORY -> VDD
- C17 pad 1: /VDD_MEMORY -> /RCC_OSC32_IN
- C19 pad 1: VDD -> RESET_N
- C2 pad 1: /GND_SHIELD -> +3V0
- C3 pad 1: VDD_NFC -> VDD
- C6 pad 1: RESET_N -> VDD
- C7 pad 1: /RCC_OSC32_IN -> VDD
- C8 pad 1: VDD -> /GND_SHIELD
- C9 pad 1: VDD -> VDD_NFC
- D1 pad 1: LED_N -> +5V
- D1 pad 2: /+LED -> /+VBUS
- D2 pad 1: /GND_SHIELD -> +3V0
- D2 pad 2: USB_DP_P -> Net-(D2-A)
- D3 pad 1: +5V -> /GND_SHIELD
- D3 pad 2: /+VBUS -> USB_DP
- D4 pad 1: +3V0 -> LED_N
- D4 pad 2: Net-(D4-A) -> /+LED
- R10 pad 1: GND -> VDD
- R10 pad 2: /BOOT0 -> I2C1_SCL_SENS
- R12 pad 1: +5V -> VDD_NFC
- R12 pad 2: USB_VBUS_SENSE_WKUP2 -> I2C2_SCL_NFC
- R2 pad 1: NFC_INT_WKUP -> GND
- R2 pad 2: VDD -> /CC2
- R3 pad 1: VDD -> +5V
- R3 pad 2: I2C1_SCL_SENS -> USB_VBUS_SENSE_WKUP2
- R6 pad 1: GND -> NFC_INT_WKUP
- R6 pad 2: /CC2 -> VDD
- R7 pad 1: VDD -> /QSPI_NCS_N
- R7 pad 2: I2C1_SDA_SENS -> /VDD_MEMORY
- R9 pad 1: GND -> VDD
- R9 pad 2: /CC1 -> I2C1_SDA_SENS
- TP1 pad 1: NFC_INT_WKUP -> GND
- TP2 pad 1: I2C1_SCL_SENS -> NFC_INT_WKUP
- TP5 pad 1: I2C1_SDA_SENS -> I2C2_SDA_NFC
- TP6 pad 1: GND -> I2C2_SCL_NFC
- U1 pad 1: /QSPI_NCS_N -> +5V
- U1 pad 2: /QSPI_IO1 -> GND
- U1 pad 3: /QSPI_IO2 -> +5V
- U1 pad 4: GND -> unconnected-(U1-NC-Pad4)
- U1 pad 5: /QSPI_IO0 -> Net-(D2-A)
- U2 pad 1: I2C1_SCL_SENS -> unconnected-(U2-V_EH-Pad1)
- U2 pad 2: unconnected-(U4-~{CS}-Pad2) -> Net-(U2-AC0)
- U2 pad 3: unconnected-(U4-SA0/SDO-Pad3) -> Net-(U2-AC1)
- U2 pad 4: I2C1_SDA_SENS -> GND
- U2 pad 5: GND -> I2C2_SDA_NFC
- U2 pad 6: GND -> I2C2_SCL_NFC
- U2 pad 7: GND -> NFC_INT_WKUP
- U2 pad 8: GND -> VDD_NFC
- U3 pad 1: unconnected-(U1-V_EH-Pad1) -> VDD
- U3 pad 2: Net-(U1-AC0) -> VDD
- U3 pad 3: Net-(U1-AC1) -> GND
- U3 pad 4: GND -> I2C1_SCL_SENS
- U3 pad 5: I2C2_SDA_NFC -> LIGHT_INT_N
- U3 pad 6: I2C2_SCL_NFC -> I2C1_SDA_SENS
- U3 pad 7: NFC_INT_WKUP -> GND
- U5 pad 1: VDD -> I2C1_SCL_SENS
- U5 pad 2: VDD -> unconnected-(U5-~{CS}-Pad2)
- U5 pad 3: GND -> unconnected-(U5-SA0/SDO-Pad3)
- U5 pad 4: I2C1_SCL_SENS -> I2C1_SDA_SENS
- U5 pad 5: LIGHT_INT_N -> GND
- U5 pad 6: I2C1_SDA_SENS -> GND
- U6 pad 1: /VDD_MEMORY -> /QSPI_NCS_N
- U6 pad 2: GND -> /QSPI_IO1
- U6 pad 3: /MEMORY_EN -> /QSPI_IO2
- U6 pad 4: VDD -> GND
- U6 pad 5: GND -> /QSPI_IO0
- U6 pad 6: unconnected-(U7-NC-Pad6) -> /QSPI_CLK
- U7 pad 1: +5V -> VDD
- U7 pad 2: GND -> USB_VBUS_SENSE_WKUP2
- U7 pad 3: +5V -> /RCC_OSC32_IN
- U7 pad 4: unconnected-(U5-NC-Pad4) -> /RCC_OSC32_OUT
- U7 pad 5: Net-(D4-A) -> unconnected-(U7-PH0-Pad5)
- U8 pad 1: unconnected-(U8-VBAT-Pad1) -> /VDD_MEMORY
- U8 pad 2: USB_VBUS_SENSE_WKUP2 -> GND
- U8 pad 3: /RCC_OSC32_IN -> /MEMORY_EN
- U8 pad 4: /RCC_OSC32_OUT -> VDD
- U8 pad 5: unconnected-(U8-PH0-Pad5) -> GND
Routing:
- net SDA: track 59.0 -> 0.00 mm, vias 2 -> 0
- net SCL: track 46.7 -> 0.00 mm, vias 2 -> 0
- net I2C1_SCL_SENS: track 0.00 -> 44.2 mm, vias 0 -> 4
- net I2C2_SDA_NFC: track 0.00 -> 42.8 mm, vias 0 -> 2
- net I2C2_SCL_NFC: track 0.00 -> 37.9 mm, vias 0 -> 2
- net I2C1_SDA_SENS: track 0.00 -> 34.0 mm, vias 1 -> 4
- net VDD_NFC: track 0.00 -> 34.0 mm, vias 0 -> 2
- net RESET_N: track 0.00 -> 31.0 mm, vias 0 -> 2
- net GND: track 37.6 -> 11.1 mm, vias 46 -> 65
- net USB_VBUS_SENSE_WKUP2: track 0.00 -> 24.3 mm, vias 0 -> 2
- net NFC_INT_WKUP: track 0.00 -> 23.9 mm, vias 0 -> 2
- net _LIGHT_INT: track 23.7 -> 0.00 mm, vias 2 -> 0
- net _NFC_INT: track 23.3 -> 0.00 mm, vias 1 -> 0
- net _RESET: track 21.3 -> 0.00 mm, vias 2 -> 0
- net TEMPRESET_N: track 0.00 -> 21.1 mm, vias 0 -> 2
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- removed copper zone on F.Cu, net VDD
Other:
- board size 55 x 45 mm -> 60 x 45 mm
- board text added: "REV 2.0.0"
- board text removed: "+3V"
- board text removed: "+5V GND"
- board text removed: "+X -X"
- board text removed: "+Y-Y"
- board text removed: "0.0000 mm / 0.0000 mm"
- board text removed: "0.3000 mm"
- board text removed: "1.6000 mm"
- board text removed: "2"
- board text removed: "55.0000 mm x 45.0000 mm"
- board text removed: "BOARD CHARACTERISTICS"
- board text removed: "Board Thickness:"
- board text removed: "Board overall dimensions:"
- board text removed: "Castellated pads:"
- board text removed: "Copper Finish:"
- board text removed: "Copper Layer Count:"
- board text removed: "Edge card connectors:"
- board text removed: "GND"
- board text removed: "Impedance Control:"
- board text removed: "Min hole diameter:"
- board text removed: "Min track/spacing:"
- board text removed: "NFC_INT"
- board text removed: "No"
- board text removed: "None"
- board text removed: "Plated Board Edge:"
- board text removed: "REV 1.0.0"
- board text removed: "SCL"
- board text removed: "SDA"
- board text removed: "TP: NFC_INT SCL SDA"
